File: Relay1.sch (KiCad schematic (older format))
At the start: 4 parts, among them Q1 BC548BTA

Commit message: rev 1a, XO fixed, more labels and rearranging
Parts:
- Q1: symbol dk_Transistors-Bipolar-BJT-Single:BC548BTA -> arduBell-rescue:BC548BTA-dk_Transistors-Bipolar-BJT-Single
- RLY1: symbol dk_Signal-Relays-Up-to-2-Amps:HJR-4102 -> arduBell-rescue:HJR-4102-dk_Signal-Relays-Up-to-2-Amps
Changed lines of the file:
@@
 $Descr A4 11693 8268
 encoding utf-8
-Sheet 2 6
+Sheet 3 6
 Title ""
 Date ""
@@
 AR Path="/6027EA0A/60283B0E" Ref="D2"  Part="1"
 AR Path="/6043B5CC/60283B0E" Ref="D1"  Part="1"
-F 0 "D2" V 1954 2170 50  0000 L CNN
+F 0 "D1" V 1954 2170 50  0000 L CNN
 F 1 "D_Small" V 2045 2170 50  0000 L CNN
 F 2 "Diode_THT:D_DO-34_SOD68_P7.62mm_Horizontal" V 2000 2100 50  0001 C CNN
@@
 AR Path="/6027EA0A/60283B18" Ref="#PWR0115"  Part="1"
 AR Path="/6043B5CC/60283B18" Ref="#PWR0116"  Part="1"
-F 0 "#PWR0115" H 2500 3050 50  0001 C CNN
+F 0 "#PWR0116" H 2500 3050 50  0001 C CNN
 F 1 "GND" H 2505 3127 50  0000 C CNN
 F 2 "" H 2500 3300 50  0001 C CNN
@@
 in
 $Comp
-L dk_Signal-Relays-Up-to-2-Amps:HJR-4102 RLY1
+L arduBell-rescue:HJR-4102-dk_Signal-Relays-Up-to-2-Amps RLY1
 U 1 1 60290BC2
 P 2700 2100
 AR Path="/6027EA0A/60290BC2" Ref="RLY1"  Part="1"
 AR Path="/6043B5CC/60290BC2" Ref="RLY2"  Part="1"
-F 0 "RLY1" H 3028 2146 50  0000 L CNN
+F 0 "RLY2" H 3028 2146 50  0000 L CNN
 F 1 "HJR-4102" H 3028 2055 50  0000 L CNN
 F 2 "Relay_THT:Relay_SPDT_HJR-4102" H 2900 2300 50  0001 L CNN
@@
 AR Path="/6027EA0A/604366B5" Ref="#PWR0114"  Part="1"
 AR Path="/6043B5CC/604366B5" Ref="#PWR0117"  Part="1"
-F 0 "#PWR0114" H 3150 1450 50  0001 C CNN
+F 0 "#PWR0117" H 3150 1450 50  0001 C CNN
 F 1 "GND" H 3155 1527 50  0000 C CNN
 F 2 "" H 3150 1700 50  0001 C CNN
@@
 	2800 2500 2900 2500
 $Comp
-L dk_Transistors-Bipolar-BJT-Single:BC548BTA Q1
+L arduBell-rescue:BC548BTA-dk_Transistors-Bipolar-BJT-Single Q1
 U 1 1 604A517E
 P 2400 3000
 AR Path="/6027EA0A/604A517E" Ref="Q1"  Part="1"
 AR Path="/6043B5CC/604A517E" Ref="Q2"  Part="1"
-F 0 "Q1" H 2588 3053 60  0000 L CNN
+F 0 "Q2" H 2588 3053 60  0000 L CNN
 F 1 "BC548BTA" H 2588 2947 60  0000 L CNN
 F 2 "Package_TO_SOT_THT:TO-92L_Inline" H 2600 3200 60  0001 L CNN
@@
 AR Path="/6027EA0A/604A7A45" Ref="R10"  Part="1"
 AR Path="/6043B5CC/604A7A45" Ref="R11"  Part="1"
-F 0 "R10" V 1854 3000 50  0000 C CNN
+F 0 "R11" V 1854 3000 50  0000 C CNN
 F 1 "1k" V 1945 3000 50  0000 C CNN
 F 2 "Resistor_SMD:R_0603_1608Metric" H 2050 3000 50  0001 C CNN
@@
 AR Path="/6027EA0A/604A9A56" Ref="#PWR0123"  Part="1"
 AR Path="/6043B5CC/604A9A56" Ref="#PWR0124"  Part="1"
-F 0 "#PWR0123" H 2500 1400 50  0001 C CNN
+F 0 "#PWR0124" H 2500 1400 50  0001 C CNN
 F 1 "VCC" H 2515 1723 50  0000 C CNN
 F 2 "" H 2500 1550 50  0001 C CNN
